File: eagle/AVC-LAN-2.brd (EAGLE design)
At the start: 88.8 x 51.8 mm, 26 parts, among them IC1 MEGA8-AI, IC3 LTC485S, IC4 MCP1825S, Q1 CSTCR12M0G, X1 1501_03

Commit message: Small update to .gitignore and added correct RS485 driver part
Parts:
- IC3: value LTC485S -> SN75HVD11D
Changed lines of the file:
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@@
 <element name="C2" library="rcl-2" package="C0603" value=".1uF" x="45.847" y="33.274" rot="R180"/>
 <element name="C3" library="rcl-2" package="C0603" value=".1uF" x="26.035" y="32.893" rot="R180"/>
-<element name="IC3" library="linear-technology" package="SOIC8" value="LTC485S" x="33.147" y="28.956" rot="R90">
+<element name="IC3" library="linear-technology" package="SOIC8" value="SN75HVD11D" x="33.147" y="28.956" rot="R90">
 <attribute name="OC_NEWARK" value="unknown" x="52.197" y="58.166" size="1.778" layer="27" rot="R90" display="off"/>
 <attribute name="MPN" value="" x="52.197" y="58.166" size="1.778" layer="27" rot="R90" display="off"/>
