File: eagle/AVC-LAN-2.sch (EAGLE design)
At the start: 26 parts, among them IC1 MEGA8-AI, IC3 LTC485S, IC4 MCP1825S, Q1 CSTCR12M0G, X1 1501_03

Commit message: Small update to .gitignore and added correct RS485 driver part
Parts:
- IC3: value LTC485S -> SN75HVD11D
Changed lines of the file:
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@@
 <part name="GND6" library="supply1" deviceset="GND" device=""/>
 <part name="GND7" library="supply1" deviceset="GND" device=""/>
-<part name="IC3" library="linear-technology" deviceset="LTC485" device="S"/>
+<part name="IC3" library="linear-technology" deviceset="LTC485" device="S" value="SN75HVD11D"/>
 <part name="V2" library="supply0" deviceset="+3V3" device=""/>
 <part name="V3" library="supply0" deviceset="+3V3" device=""/>
